File: controller-board/controller-board.kicad_pcb (KiCad board)
At the start: 2 copper layers, 24.2 x 42.8 mm, 14 parts, among them J1 22057025, J2 22057035, J3 DF40B-10DS-0.4V_58_, SW2 B3F-3152, U1 ATtiny4-MA, U2 ADG1236YCPZ-REEL7, U3 TLV709A33DBVR

Commit message: updated README.md & image added
Parts:
- moved J2 7.25 mm to (132.4, 58.9), turned to 180 degrees
- moved J1 5.77 mm to (119.3, 58.9), turned to 180 degrees
Routing:
- net -15V: track 16.0 -> 9.73 mm
- net +15V: track 25.0 -> 30.9 mm
- net PB1: track 48.0 -> 44.2 mm
