File: controller-board/controller-board.kicad_sch (KiCad schematic)
At the start: 14 parts, among them J1 22057025, J2 22057035, J3 DF40B-10DS-0.4V_58_, SW2 B3F-3152, U1 ATtiny4-MA, U2 ADG1236YCPZ-REEL7, U3 TLV709A33DBVR

Commit message: updated README.md & image added
Other:
- note added: "For Program/Debug ATtimy"
- note added: "Replacement of Original Channel Switch"
- moved on the sheet: C1, C2, C3, C4, C6, D1, J1, J2, J3, SW1A, SW1B, SW2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
