File: power-board/power_board.kicad_pcb (KiCad board)
At the start: 2 copper layers, 13.9 x 29.6 mm, 7 parts, among them J1 Conn_01x01_Pin, J2 Conn_01x01_Pin, J3 Conn_01x01_Pin, J4 Conn_01x01_Pin, J5 22057035

Commit message: updated README.md & image added
Parts:
- J1, J2, J3, J4: moved to B.Cu
- moved J5 7.35 mm to (154.4, 74.4), turned to 180 degrees
- turned J1 to 180 degrees
- turned J2 to 180 degrees
- turned J3 to 180 degrees
- turned J4 to 180 degrees
Routing:
- net -15V: track 17.4 -> 10.4 mm
- net +15V: track 17.3 -> 10.6 mm
